File: Eagle/MOC/moc.sch (EAGLE design)
At the start: 33 parts, among them IC2 74HC595N, IC3 74HC595N, IC4 74HC595N, IC6 MEGA8-P, IC7 7805TV, K1 4052, Q1 20MHz

Commit message: hardware tests, all features
Parts:
- removed C10, C9: (no value), resistor:C-EU025-025X050
- removed C5: (no value), resistor:CPOL-EUE2.5-7
- removed C8: 100n, resistor:C-EU025-025X050
- removed IC4: 74HC595N, 74xx-eu:74HC595N
- removed L1: (no value), resistor:L-EU0207/10
- removed Q1: 20MHz, crystal:CRYSTALHC49S
- added H1, H2, H3, H4, H5, H6: MOUNT-HOLE3.2, holes:MOUNT-HOLE3.2
- added JP10: (no value), pinhead:PINHD-1X3
- added JP11: (no value), pinhead:PINHD-1X2/90
- added JP2: HV_MODULE, pinhead:PINHD-1X2
- added JP3: M_SW, pinhead:PINHD-1X2/90
- added JP7: H_SW, pinhead:PINHD-1X2/90
- added JP8: (no value), pinhead:PINHD-1X8
- added JP9: prog, pinhead:PINHD-1X3
- C12: device resistor:CPOL-EUE2.5-7 -> resistor:CPOL-EUE3.5-8
- IC7: value 7805TV -> 7805T; device linear:7805TV -> linear:7805T
- JP1: device pinhead:PINHD-1X30 -> pinhead:PINHD-1X8
- JP4: value (none) -> DS3231_POWER
- JP5: value (none) -> DS3231_SIGNALS
- JP6: value (none) -> RELAY_MODE
- R43: device resistor:R-EU_0207/7 -> resistor:R-EU_0207/10
- R44, R45: device resistor:R-EU_0204/5 -> resistor:R-EU_0207/10
- R47: device resistor:R-EU_0204/2V -> resistor:R-EU_0207/10
Connections:
- removed net D0: IC4A.QH, JP1.24
- removed net D1: IC4A.QG, JP1.23
- removed net D2: IC4A.QF, JP1.22
- removed net D3: JP1.21
- removed net D4: IC4A.QD, IC4A.QE, JP1.20
- removed net D5: IC4A.QC, JP1.19
- removed net D6: IC4A.QB, JP1.18
- removed net D7: IC4A.QA, JP1.17
- removed net HV: JP1.30
- removed net N$41: C9.2, IC6.PB6(XTAL1/TOSC1), Q1.2
- removed net N$42: C10.2, IC6.PB7(XTAL2/TOSC2), Q1.1
- removed net N$52: C8.2, IC6.AVCC, L1.1
- removed net N$56: IC6.PC6(/RESET), R47.1
- removed net S_IN: IC4A.SER, IC6.PB4(MISO)
- removed net VCC: IC2A.SCL, IC3A.SCL, IC4A.SCL
- new net H_CH: IC6.PB1(OC1A), JP7.1
- new net MISO: IC6.PB4(MISO), JP9.2
- new net M_CH: IC6.PB0(ICP), JP3.1
- new net NEON: IC6.PD7(AIN1), JP10.3
- new net RESET: IC6.PC6(/RESET), JP11.1, R47.1
- net +12V: now also JP2.1
- net +5V: now also IC2A.SCL, IC3A.SCL, IC6.AVCC, JP10.1; no longer C5.+, IC4P.VCC, JP1.26, L1.2
- net D10: now also JP8.6; no longer JP1.14
- net D11: now also JP8.5; no longer JP1.13
- net D12: now also JP8.4; no longer JP1.12
- net D13: now also JP8.3; no longer JP1.11
- net D14: now also JP8.2; no longer JP1.10
- net D15: now also JP8.1; no longer JP1.9
- net D8: now also JP8.8; no longer JP1.16
- net D9: now also JP8.7; no longer JP1.15
- net GND: now also JP10.2, JP11.2, JP2.2, JP3.2, JP7.2; no longer C10.1, C5.-, C8.1, C9.1, IC4A.G, IC4P.GND, JP1.25
- net H_IN: now also IC6.PC2(ADC2); no longer IC6.PC0(ADC0)
- net IN_CLK: now also IC6.PC1(ADC1); no longer IC4A.SCK, IC6.PB3(MOSI/OC2)
- net MODE_0: now also IC6.PB3(MOSI/OC2), JP9.1; no longer IC6.PD0(RXD)
- net MODE_1: now also IC6.PB2(SS/OC1B); no longer IC6.PD1(TXD)
- net M_IN: now also JP9.3
- net OUT_CLK: now also IC6.PC0(ADC0); no longer IC4A.RCK, IC6.PB2(SS/OC1B)
- net RELAY: now also IC6.PD0(RXD); no longer IC6.PC3(ADC3)
- net SQW: now also IC6.PC3(ADC3); no longer IC6.PC1(ADC1)
Other:
- note added: "Switches"

Commit message: cathodes heat on mode, relay parameters
Parts:
- JP3, JP7: device pinhead:PINHD-1X2/90 -> pinhead:PINHD-1X2
- JP6: device pinhead:PINHD-1X3/90 -> pinhead:PINHD-1X3
Changed lines of the file:
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@@
 <part name="P+1" library="supply1" library_urn="urn:adsk.eagle:library:371" deviceset="+5V" device=""/>
 <part name="P+2" library="supply1" library_urn="urn:adsk.eagle:library:371" deviceset="+5V" device=""/>
-<part name="JP6" library="pinhead" library_urn="urn:adsk.eagle:library:325" deviceset="PINHD-1X3" device="/90" package3d_urn="urn:adsk.eagle:package:22459/2" value="RELAY_MODE"/>
+<part name="JP6" library="pinhead" library_urn="urn:adsk.eagle:library:325" deviceset="PINHD-1X3" device="" package3d_urn="urn:adsk.eagle:package:22458/2" value="RELAY_MODE"/>
 <part name="GND1" library="supply1" library_urn="urn:adsk.eagle:library:371" deviceset="GND" device=""/>
 <part name="JP2" library="pinhead" library_urn="urn:adsk.eagle:library:325" deviceset="PINHD-1X2" device="" package3d_urn="urn:adsk.eagle:package:22435/2" value="HV_MODULE"/>
 <part name="P+8" library="supply1" library_urn="urn:adsk.eagle:library:371" deviceset="+12V" device=""/>
-<part name="JP3" library="pinhead" library_urn="urn:adsk.eagle:library:325" deviceset="PINHD-1X2" device="/90" package3d_urn="urn:adsk.eagle:package:22437/2" value="M_SW"/>
-<part name="JP7" library="pinhead" library_urn="urn:adsk.eagle:library:325" deviceset="PINHD-1X2" device="/90" package3d_urn="urn:adsk.eagle:package:22437/2" value="H_SW"/>
+<part name="JP3" library="pinhead" library_urn="urn:adsk.eagle:library:325" deviceset="PINHD-1X2" device="" package3d_urn="urn:adsk.eagle:package:22435/2" value="M_SW"/>
+<part name="JP7" library="pinhead" library_urn="urn:adsk.eagle:library:325" deviceset="PINHD-1X2" device="" package3d_urn="urn:adsk.eagle:package:22435/2" value="H_SW"/>
 <part name="GND3" library="supply1" library_urn="urn:adsk.eagle:library:371" deviceset="GND" device=""/>
 <part name="JP1" library="pinhead" library_urn="urn:adsk.eagle:library:325" deviceset="PINHD-1X8" device="" package3d_urn="urn:adsk.eagle:package:22409/2"/>
